Commit message: Included Robot Model in the tutorial

File: robair_description/urdf/robair.urdf.xacro (robot description, xacro)
@@ -9,5 +9,6 @@
   <!-- ######################### Links ############################### -->
   <!-- base_link -->
-  <link name="base_link"></link>
+  <link name="$(arg parent)"></link>
+  <!-- <link name="base_link"></link> -->
   <!-- body -->
   <xacro:property name="height" value="0.2" />
@@ -21,5 +22,5 @@
           </geometry>
               <material name="Cyan">
-              <color rgba="0 1.0 1.0 0.3"/>
+              <color rgba="0 1.0 1.0 0.7"/>
           </material>
           </visual>
@@ -54,9 +55,9 @@
   <!-- ########## Joints ################### -->
   <joint name="base_link_to_body" type="fixed">
-    <parent link="base_link"/>
+    <parent link="$(arg parent)"/>
     <child link="body"/>
-    <origin xyz="0 0 0" rpy="0 0 0"/>
+    <origin xyz="0 0 -0.22" rpy="0 0 0"/>
   </joint>
-  <joint name="left_wheel" type="continuous">
+  <joint name="left_wheel" type="fixed"> <!-- type="continuous" -->
     <parent link="body"/>
     <child link="left_wheel_link"/>
@@ -64,5 +65,5 @@
     <axis xyz="0 1 0" rpy="0 0 0" />
   </joint>
-  <joint name="right_wheel" type="continuous">
+  <joint name="right_wheel" type="fixed"> <!-- type="continuous" -->
     <parent link="body"/>
     <child link="right_wheel_link"/>
@@ -82,5 +83,5 @@
     <axis xyz="1 0 0" rpy="0 0 0" />
   </joint>
-  <joint name="front_wheel" type="fixed">
+  <joint name="front_wheel" type="fixed"> <!-- type="continuous" -->
     <parent link="front_wheel_support"/>
     <child link="front_wheel_link"/>
@@ -88,5 +89,5 @@
     <axis xyz="0 0.0 0.0" rpy="0 0 0" />
   </joint>
-  <joint name="rear_wheel" type="fixed">
+  <joint name="rear_wheel" type="fixed"> <!-- type="continuous" -->
     <parent link="rear_wheel_support"/>
     <child link="rear_wheel_link"/>

Commit message: Update Visualization

File: robair_description/urdf/robair.urdf.xacro (robot description, xacro)
@@ -57,5 +57,5 @@
     <parent link="$(arg parent)"/>
     <child link="body"/>
-    <origin xyz="0 0 -0.22" rpy="0 0 0"/>
+    <origin xyz="-0.25 0 -0.22" rpy="0 0 0"/>
   </joint>
   <joint name="left_wheel" type="fixed"> <!-- type="continuous" -->

Commit message: fix joints names and type

File: robair_description/urdf/robair.urdf.xacro (robot description, xacro)
@@ -59,5 +59,5 @@
     <origin xyz="-0.25 0 -0.22" rpy="0 0 0"/>
   </joint>
-  <joint name="left_wheel" type="fixed"> <!-- type="continuous" -->
+  <joint name="left_wheel" type="fixed"> <!-- type="continuous/fixed" -->
     <parent link="body"/>
     <child link="left_wheel_link"/>
@@ -65,5 +65,5 @@
     <axis xyz="0 1 0" rpy="0 0 0" />
   </joint>
-  <joint name="right_wheel" type="fixed"> <!-- type="continuous" -->
+  <joint name="right_wheel" type="fixed"> <!-- type="continuous/fixed" -->
     <parent link="body"/>
     <child link="right_wheel_link"/>
@@ -83,5 +83,5 @@
     <axis xyz="1 0 0" rpy="0 0 0" />
   </joint>
-  <joint name="front_wheel" type="fixed"> <!-- type="continuous" -->
+  <joint name="front_wheel" type="fixed"> <!-- type="continuous/fixed" -->
     <parent link="front_wheel_support"/>
     <child link="front_wheel_link"/>
@@ -89,5 +89,5 @@
     <axis xyz="0 0.0 0.0" rpy="0 0 0" />
   </joint>
-  <joint name="rear_wheel" type="fixed"> <!-- type="continuous" -->
+  <joint name="rear_wheel" type="fixed"> <!-- type="continuous/fixed" -->
     <parent link="rear_wheel_support"/>
     <child link="rear_wheel_link"/>
