Commit message: Update readme.md

File: robair_description/urdf/wheel.urdf.xacro (robot description, xacro)
@@ -36,8 +36,9 @@
 				</geometry>
 			</visual>
+			<!-- TODO: collision description to be fixed! -->
 			<collision>
 				<origin xyz="0 0 0" rpy="${M_PI/2} 0 0" />
 				<geometry>
-					<cylinder length="${wheel_length}" radius="${wheel_radius}" />
+					<cylinder length="${wheel_length}" radius="${wheel_radius/3}" />
 				</geometry>
 			</collision>
