Commit message: Update Gazebo Simulation

File: robair_description/urdf/caster_wheel.urdf.xacro (robot description, xacro)
@@ -28,5 +28,4 @@
         <child link="${prefix}_caster_wheel_link"/>
         <xacro:insert_block name="origin"/>
-        <axis xyz="0 1 0" rpy="0 0 0" />
     </joint>
   </xacro:macro>

File: robair_description/urdf/robair.urdf.xacro (robot description, xacro)
@@ -13,19 +13,23 @@
   <xacro:property name="width"  value="0.3" />
   <link name="robair_body">
-      <visual>
-          <origin xyz="0 0 0.1" rpy="0 0 0" />
-          <geometry>
-              <box size="${length} ${width} ${height}"/>
-          </geometry>
-              <material name="Cyan">
-                <color rgba="0 1.0 1.0 0.7"/>
-              </material>
-          </visual>
-      <collision>
-          <origin xyz="0 0 0.1" rpy="0 0 0" />
-          <geometry>
-              <box size="${length} ${width} ${height}"/>
-          </geometry>
-      </collision>
+    <inertial>
+      <mass value="10"/>
+      <inertia ixx="0.4" ixy="0.0" ixz="0.0" iyy="0.4" iyz="0.0" izz="0.2"/>
+    </inertial>
+    <visual>
+      <origin xyz="0 0 0.1" rpy="0 0 0" />
+      <geometry>
+          <box size="${length} ${width} ${height}"/>
+      </geometry>
+      <material name="Cyan">
+        <color rgba="0 1.0 1.0 0.7"/>
+      </material>
+    </visual>
+    <collision>
+        <origin xyz="0 0 0.1" rpy="0 0 0" />
+        <geometry>
+            <box size="${length} ${width} ${height}"/>
+        </geometry>
+    </collision>
   </link>
   <!-- Wheel Mounting Positions -->
