Commit message: Update Launch files

File: robair_description/urdf/hokuyo.urdf.xacro (robot description, xacro)
@@ -64,4 +64,12 @@
         <material name="black" />
       </visual>
+      <collision>
+        <origin xyz="0.0 0 0.24" rpy="0 0 0" />
+        <geometry>
+          <!-- Origin of this mesh is the base of the bracket. -->
+          <cylinder length="0.08" radius="0.03" />
+        </geometry>
+        <material name="black" />
+      </collision>
     </link>
     <joint name="${prefix}_laser_joint" type="fixed">

File: robair_description/urdf/robair.urdf.xacro (robot description, xacro)
@@ -6,14 +6,11 @@
   <xacro:include filename="$(find robair_description)/urdf/wheel.urdf.xacro" />
   <!-- Wheel Support -->
-  <xacro:include filename="$(find robair_description)/urdf/wheel_support.urdf.xacro" />
+  <xacro:include filename="$(find robair_description)/urdf/caster_wheel.urdf.xacro" />
   <!-- ######################### Links ############################### -->
-  <!-- base_link -->
-  <link name="$(arg parent)"></link>
-  <!-- <link name="base_link"></link> -->
-  <!-- body -->
+  <!-- robair_body -->
   <xacro:property name="height" value="0.2" />
   <xacro:property name="length" value="0.5" />
   <xacro:property name="width"  value="0.3" />
-  <link name="body">
+  <link name="robair_body">
       <visual>
           <origin xyz="0 0 0.1" rpy="0 0 0" />
@@ -22,8 +19,9 @@
           </geometry>
               <material name="Cyan">
-              <color rgba="0 1.0 1.0 0.7"/>
-          </material>
+                <color rgba="0 1.0 1.0 0.7"/>
+              </material>
           </visual>
       <collision>
+          <origin xyz="0 0 0.1" rpy="0 0 0" />
           <geometry>
               <box size="${length} ${width} ${height}"/>
@@ -33,69 +31,29 @@
   <!-- Wheel Mounting Positions -->
   <xacro:property name="wheel_vertical_offset" value="0.01" />
-  <!-- ROBAIR wheel macros -->
+  <!-- ROBAIR wheels macros -->
+  <xacro:wheel wheel_prefix="right" wheel_length="0.02" wheel_radius="0.5">
+    <origin xyz="0 ${0.024 + width/2} ${wheel_vertical_offset}" rpy="0 0 0" />
+  </xacro:wheel>
   <xacro:wheel wheel_prefix="left" wheel_length="0.02" wheel_radius="0.5">
-    <origin xyz="0 ${-length/2} ${wheel_vertical_offset}" rpy="0 0 0" />
+    <origin xyz="0 ${-0.024-width/2} ${wheel_vertical_offset}" rpy="0 0 0" />
   </xacro:wheel>
-  <xacro:wheel wheel_prefix="right" wheel_length="0.02" wheel_radius="0.5">
-    <origin xyz="0 ${length/2} ${wheel_vertical_offset}" rpy="0 0 0" />
-  </xacro:wheel>
-  <xacro:wheel wheel_prefix="front" wheel_length="0.01" wheel_radius="0.3">
-    <origin xyz="0 0 0" rpy="0 0 0" />
-  </xacro:wheel>
-  <xacro:wheel wheel_prefix="rear" wheel_length="0.01" wheel_radius="0.3">
-    <origin xyz="0 0 0" rpy="0 0 0" />
-  </xacro:wheel>
-  <!-- ROBAIR Wheel Supports -->
-  <xacro:wheel_support prefix="front">
-    <origin xyz="0 0 ${wheel_vertical_offset}" rpy="0 0 0" />
-  </xacro:wheel_support>
-  <xacro:wheel_support prefix="rear">
-    <origin xyz="0 0 ${wheel_vertical_offset}" rpy="0 0 0" />
-  </xacro:wheel_support>
+  <!-- Caster Wheels -->
+  <xacro:caster_wheel prefix="front">
+    <origin xyz="${-0.1+length/2} 0 ${wheel_vertical_offset}" rpy="0 0 0" />
+  </xacro:caster_wheel>
+  <xacro:caster_wheel prefix="rear">
+    <origin xyz="${+0.1-length/2} 0 ${wheel_vertical_offset}" rpy="0 0 0" />
+  </xacro:caster_wheel>
   <!-- ########## Joints ################### -->
-  <joint name="base_link_to_body" type="fixed">
+  <!-- base_link -->
+  <link name="$(arg parent)"></link>
+  <joint name="parent_to_robair_body_joint" type="fixed">
     <parent link="$(arg parent)"/>
-    <child link="body"/>
+    <child link="robair_body"/>
     <origin xyz="-0.25 0 -0.22" rpy="0 0 0"/>
-  </joint>
-  <joint name="left_wheel" type="fixed"> <!-- type="continuous/fixed" -->
-    <parent link="body"/>
-    <child link="left_wheel_link"/>
-    <origin xyz="0 ${-length/3} ${wheel_vertical_offset}" rpy="0 0 0" />
-    <axis xyz="0 1 0" rpy="0 0 0" />
-  </joint>
-  <joint name="right_wheel" type="fixed"> <!-- type="continuous/fixed" -->
-    <parent link="body"/>
-    <child link="right_wheel_link"/>
-    <origin xyz="0 ${length/3} ${wheel_vertical_offset}" rpy="0 0 0" />
-    <axis xyz="0 1 0" rpy="0 0 0" />
-  </joint>
-  <joint name="front_support_joint" type="fixed">
-    <parent link="body" />
-    <child link="front_wheel_support" />
-    <origin xyz="${width/2} -0.032 ${wheel_vertical_offset/2}" rpy="0 0 0" />
-    <axis xyz="1 0 0" rpy="0 0 0" />
-  </joint>
-  <joint name="rear_support_joint" type="fixed">
-    <parent link="body" />
-    <child link="rear_wheel_support" />
-    <origin xyz="${-width/2} -0.032 ${wheel_vertical_offset/2}" rpy="0 0 0" />
-    <axis xyz="1 0 0" rpy="0 0 0" />
-  </joint>
-  <joint name="front_wheel" type="fixed"> <!-- type="continuous/fixed" -->
-    <parent link="front_wheel_support"/>
-    <child link="front_wheel_link"/>
-    <origin xyz="0.05 0.03 -0.01" rpy="0 0 0" />
-    <axis xyz="0 0.0 0.0" rpy="0 0 0" />
-  </joint>
-  <joint name="rear_wheel" type="fixed"> <!-- type="continuous/fixed" -->
-    <parent link="rear_wheel_support"/>
-    <child link="rear_wheel_link"/>
-    <origin xyz="0.05 0.03 -0.01" rpy="0 0 0" />
-    <axis xyz="0 0.0 0.0" rpy="0 0 0" />
   </joint>
   <!-- ### Laser Sensor Activation -->
   <!-- Laser Scanner Placement and Parameters -->
-  <xacro:arg name="laser_ust10_parent"  default="$(optenv ROBAIR_UST10_PARENT body)" />
+  <xacro:arg name="laser_ust10_parent"  default="$(optenv ROBAIR_UST10_PARENT robair_body)" />
   <xacro:arg name="laser_ust10_topic"   default="$(optenv ROBAIR_UST10_TOPIC /scan)" />
   <xacro:arg name="laser_ust10_xyz"     default="$(optenv ROBAIR_UST10_XYZ 0.2206 0.0 0.0)" />
@@ -104,9 +62,9 @@
     <origin xyz="$(arg laser_ust10_xyz)" rpy="$(arg laser_ust10_rpy)" />
   </xacro:hokuyo_ust10_mount>
-  <!-- Interface with ros control -->
-  <!-- <gazebo>
+  <!-- Interface with Gazebo ros control -->
+  <gazebo>
     <plugin name="gazebo_ros_control" filename="libgazebo_ros_control.so">
-      <robotNamespace>/</robotNamespace>
+      <robotNamespace>/robair</robotNamespace>
     </plugin>
-  </gazebo> -->
+  </gazebo>
 </robot>

File: robair_description/urdf/wheel.urdf.xacro (robot description, xacro)
@@ -21,5 +21,5 @@
 ARISING IN ANY WAY OUT OF THE USE OF THIS SOFTWARE, EVEN IF ADVISED OF THE POSSIBILITY OF SUCH DAMAGE.-->
 <!-- Source: https://github.com/husky/husky/blob/noetic-devel/husky_description/urdf/wheel.urdf.xacro -->
-<robot xmlns:xacro="http://ros.org/wiki/xacro" name="wheel">
+<robot name="wheel" xmlns:xacro="http://ros.org/wiki/xacro">
 	<xacro:property name="M_PI" value="3.14159"/>
 	<xacro:macro name="wheel" params="wheel_prefix wheel_length wheel_radius *joint_pose">
@@ -38,7 +38,7 @@
 			<!-- TODO: collision description to be fixed! -->
 			<collision>
-				<origin xyz="0 0 0" rpy="${M_PI/2} 0 0" />
+				<origin xyz="0 0 0" rpy="${-M_PI/2} 0 0" />
 				<geometry>
-					<cylinder length="${wheel_length}" radius="${wheel_radius/3}" />
+					<cylinder length="0.05" radius="0.08" />
 				</geometry>
 			</collision>
@@ -51,10 +51,10 @@
 			<fdir1 value="1 0 0"/>
 		</gazebo>
-		<!-- <joint name="${wheel_prefix}_wheel" type="continuous">
-			<parent link="body"/>
+		<joint name="${wheel_prefix}_wheel" type="continuous">
+			<parent link="robair_body"/>
 			<child link="${wheel_prefix}_wheel_link"/>
 			<xacro:insert_block name="joint_pose"/>
 			<axis xyz="0 1 0" rpy="0 0 0" />
-		</joint> -->
+		</joint>
 		<transmission name="${wheel_prefix}_wheel_trans" type="SimpleTransmission">
 			<type>transmission_interface/SimpleTransmission</type>

Commit message: fix laserscanner stl

File: robair_description/urdf/hokuyo.urdf.xacro (robot description, xacro)
@@ -60,5 +60,5 @@
         <geometry>
           <!-- Origin of this mesh is the base of the bracket. -->
-          <mesh filename="package://urg_node/meshes/hokuyo_ust10.stl" />
+          <mesh filename="package://robair_description/meshes/hokuyo_ust10.stl" />
         </geometry>
         <material name="black" />
